File: esp32.kicad_sch (KiCad schematic)
At the start: 51 parts, among them J1 USB_C_Receptacle_USB2.0_16P, J2 Micro_SD_Card, J3 AudioJack3, J4 BATTERY CONNECTOR, J5 Conn_01x04, SW3 SW_Push, SW4 SW_Push, SW5 SW_Push, U3 TP4056-42-ESOP8, U4 PCM5102A, U5 TPS61022, U6 ESP32-WROOM-32

Commit message: removed the battery and its components and added the new revised power regulation with correct current ratings and made it minimalistic
Parts:
- removed C29: 2.2uF, Capacitor_SMD:C_0201_0603Metric, symbol Device:C
- removed C30, C31: 4.7uF, Capacitor_SMD:C_0201_0603Metric, symbol Device:C
- removed D2: 1N914, Diode_SMD:D_0603_1608Metric, symbol Diode:1N914
- removed D3, D4, D5: LED, LED_SMD:LED_0603_1608Metric, symbol Device:LED
- removed J4: BATTERY CONNECTOR, Connector_JST:JST_PH_S2B-PH-K_1x02_P2.00mm_Horizontal, symbol Connector_Generic:Conn_01x02
- removed L3: 1uH, Inductor_SMD:L_0201_0603Metric, symbol Device:L
- removed R17: 2k, Resistor_SMD:R_0201_0603Metric, symbol Device:R
- removed R18, R19, R22: 1k, Resistor_SMD:R_0201_0603Metric, symbol Device:R
- removed R20: 453k, Resistor_SMD:R_0603_1608Metric, symbol Device:R
- removed R21: 100k, Resistor_SMD:R_0603_1608Metric, symbol Device:R
- removed U3: TP4056-42-ESOP8, Package_SO:SOIC-8-1EP_3.9x4.9mm_P1.27mm_EP2.41x3.3mm_ThermalVias, symbol Battery_Management:TP4056-42-ESOP8
- removed U5: TPS61022, Package_DFN_QFN:Texas_RWU0007A_VQFN-7_2x2mm_P0.5mm, symbol Converter_DCDC:TPS61022
- added D1: LED, symbol Device:LED
- added D3: 1N5817, Diode_THT:D_DO-41_SOD81_P10.16mm_Horizontal, symbol Diode:1N5817
- added L1: L, symbol Device:L
- added R10: 100k, Resistor_SMD:R_0603_1608Metric, symbol Device:R
- added R11: 500, Resistor_SMD:R_0603_1608Metric, symbol Device:R
- added R9: 453, Resistor_SMD:R_0603_1608Metric, symbol Device:R
- added U1: TLV62569ADRL, Package_TO_SOT_SMD:SOT-563, symbol Regulator_Switching:TLV62569ADRL
- C21: value 100nF -> 10uF
- C27: value 10uF -> 4.7uF; footprint Capacitor_SMD:C_0201_0603Metric -> Capacitor_SMD:C_0603_1608Metric
- C28: value 10uF -> 22uF; footprint Capacitor_SMD:C_0201_0603Metric -> Capacitor_SMD:C_0603_1608Metric
Connections:
- net +4.2V is gone; now on net +5V: C27.1
- net +3.3V: now also C28.1, D1.2 (A), L1.2, R9.1
- net +5V: now also D3.1 (K), U1.3 (VIN), U1.5 (EN); no longer C28.1
- net GND: now also R10.2, R11.2, U1.2 (GND)
- net at J1.A4 (VBUS), J1.A9 (VBUS), J1.B4 (VBUS)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: now also D3.2 (A)
- new net: R10.1, R9.2, U1.1 (FB)
- new net: D1.1 (K), R11.1
- new net: L1.1, U1.4 (SW)
Other:
- note removed: "CHARGING CONTROLLER"
- moved on the sheet: J3, SW3, U4

Commit message: Done multiple changes here and there must for of all I routed the new parts in including the new converter for steping down power and the new smaller buttons and was able to change the board shape hahaha
Parts:
- D1: footprint (none) -> LED_SMD:LED_0201_0603Metric
- L1: footprint (none) -> Inductor_SMD:L_0201_0603Metric
- SW3, SW4, SW5: footprint Button_Switch_SMD:SW_SPST_TL3342 -> Button_Switch_SMD:SW_Tactile_SPST_NO_Straight_CK_PTS636Sx25SMTRLFS
Changed lines of the file:
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@@
 			)
 		)
-		(property "Footprint" "Button_Switch_SMD:SW_SPST_TL3342"
+		(property "Footprint" "Button_Switch_SMD:SW_Tactile_SPST_NO_Straight_CK_PTS636Sx25SMTRLFS"
 			(at 186.69 113.03 0)
 			(hide yes)
@@
 			)
 		)
-		(property "Footprint" ""
+		(property "Footprint" "Inductor_SMD:L_0201_0603Metric"
 			(at 72.39 22.86 0)
 			(hide yes)
@@
 			)
 		)
-		(property "Footprint" "Button_Switch_SMD:SW_SPST_TL3342"
+		(property "Footprint" "Button_Switch_SMD:SW_Tactile_SPST_NO_Straight_CK_PTS636Sx25SMTRLFS"
 			(at 49.53 135.89 0)
 			(hide yes)
@@
 			)
 		)
-		(property "Footprint" "Button_Switch_SMD:SW_SPST_TL3342"
+		(property "Footprint" "Button_Switch_SMD:SW_Tactile_SPST_NO_Straight_CK_PTS636Sx25SMTRLFS"
 			(at 124.46 135.89 0)
 			(hide yes)
@@
 			)
 		)
-		(property "Footprint" ""
+		(property "Footprint" "LED_SMD:LED_0201_0603Metric"
 			(at 97.79 22.86 0)
 			(hide yes)

Commit message: Added the power routing in the In2 Cu now all set to go for printing
Parts:
- L1: value L -> 1uH
Changed lines of the file:
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@@
 			)
 		)
-		(property "Value" "L"
+		(property "Value" "1uH"
 			(at 72.39 20.32 90)
 			(show_name no)

Commit message: Added a headphone amplifier signal and fixed the DAC converter connections based on the datasheet #almost blew it up
Parts:
- removed C20, C22: 100nF, Capacitor_SMD:C_0603_1608Metric, symbol Device:C
- removed C21: 10uF, Capacitor_SMD:C_0603_1608Metric, symbol Device:C
- removed C23, C24, C25: 2.2uF, Capacitor_SMD:C_0201_0603Metric, symbol Device:C
- removed C26, C33: 0.1uF, Capacitor_SMD:C_0201_0603Metric, symbol Device:C
- removed J3: AudioJack3, Connector_Audio:Jack_3.5mm_CUI_SJ1-3523N_Horizontal, symbol Connector_Audio:AudioJack3
- removed R16: 10k, Resistor_SMD:R_0603_1608Metric, symbol Device:R
- removed SW3: SW_Push, Button_Switch_SMD:SW_Tactile_SPST_NO_Straight_CK_PTS636Sx25SMTRLFS, symbol Switch:SW_Push
- removed U4: PCM5102A, Package_SO:TSSOP-20_4.4x6.5mm_P0.65mm, symbol Audio:PCM5102A
Other:
- added sheet page 2 (continuation.kicad_sch)
- note removed: "DAC CONVERTER"
- moved on the sheet: J2, R13, R14, R15
